File: rky/rky.kicad_sch (KiCad schematic)
At the start: 47 parts, among them J1 UART, J2 Li-Ion 3.7 CONN, J3 USB_C_Receptacle_USB2.0, SW1 SW_SPDT, U1 CP2102-GM, U2 SSD1306, U3 ESP8266-12E/ESP-12E, U4 LM3940IMP-3.3/NOPB, U5 TP4056

Commit message: rough pcb layout create
Parts:
- added U6: NRF24L01, Package_DFN_QFN:QFN-20-1EP_4x4mm_P0.5mm_EP2.5x2.5mm, symbol RF:NRF24L01

Commit message: schematic update
Parts:
- added C14: 4.7uf, Capacitor_SMD:C_0603_1608Metric, symbol Device:C_Polarized_Small_US
- added DRIVE2: PTS525SM15SMTR2LFS, push button:SW_PTS525SM15SMTR2LFS, symbol tactile switch:PTS525SM15SMTR2LFS
- added R12: 10k, Resistor_SMD:R_0603_1608Metric, symbol Device:R_Small_US
- DRIVE1, SELECT1: footprint tactile switch:SW_PTS525SM15SMTR2LFS -> push button:SW_PTS525SM15SMTR2LFS
Connections:
- net 3.3V: now also DRIVE2.2
- net GND: now also C14.1; no longer C12.2 (P$2), C13.2, U5.3 (GND)
- new net: DRIVE2.1, R12.2
- new net: C12.2 (P$2), C13.2, U5.3 (GND)
- new net INT_PWR_DN: C14.2, R12.1
Other:
- note added: "ESP8266 / UC"
- note added: "NRF24L01 RF TRANCEIVER"
- note added: "POWER OFF/ON"
- note added: "Vc=Vin(1-e^1/RC)"
- moved on the sheet: R2, R3, SELECT1, U6
