File: rky/rky.kicad_sch (KiCad schematic)
At the start: 60 parts, among them J1 Conn_01x02_Male, J2 Li-Ion 3.7 CONN, J3 USB_C_Receptacle_USB2.0, J4 Conn_01x04_Male, J5 Conn_02x03_Odd_Even, SW1 SW_SPDT, U2 SSD1306, U3 ESP8266-12E/ESP-12E, U4 LM3940IMP-3.3/NOPB, U5 TP4056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

Commit message: component place
 first touch component placement complete
Parts:
- U5: footprint tp4056 ftprnt:SOP127P600X175-9N -> Package_SO:SO-8_5.3x6.2mm_P1.27mm
- Y1: footprint (none) -> Crystal:Crystal_SMD_0603-4Pin_6.0x3.5mm
Connections:
- net RXD: now also J1.2 (Pin_2); no longer J1.1 (Pin_1)
- net TXD: now also J1.1 (Pin_1); no longer J1.2 (Pin_2)
- net SDA: now reaches J4.1 (Pin_1), U3.19 (IO4)
- net SCL: now reaches J4.2 (Pin_2), U3.20 (IO5)
Changed lines of the file:
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@@
+    (stroke (width 0) (type default) (color 0 0 0 0))
+  )
+  (polyline (pts (xy 17.78 15.24) (xy 17.78 81.28))
     (stroke (width 0) (type default) (color 0 0 0 0))
   )
@@
     (stroke (width 0) (type default) (color 0 0 0 0))
   )
+  (polyline (pts (xy 17.78 81.28) (xy 147.32 81.28))
+    (stroke (width 0) (type default) (color 0 0 0 0))
+  )
   (wire (pts (xy 69.088 257.556) (xy 77.851 257.556))
     (stroke (width 0) (type default) (color 0 0 0 0))
@@
   )
   (wire (pts (xy 180.213 227.965) (xy 180.213 246.126))
+    (stroke (width 0) (type default) (color 0 0 0 0))
+  )
+  (polyline (pts (xy 20.32 198.12) (xy 172.72 198.12))
     (stroke (width 0) (type default) (color 0 0 0 0))
   )
@@
     (stroke (width 0) (type default) (color 0 0 0 0))
   )
+  (polyline (pts (xy 172.72 83.82) (xy 20.32 83.82))
+    (stroke (width 0) (type default) (color 0 0 0 0))
+  )
   (wire (pts (xy 210.82 108.585) (xy 193.04 108.585))
     (stroke (width 0) (type default) (color 0 0 0 0))
@@
   )
   (polyline (pts (xy 402.336 15.24) (xy 287.401 14.986))
+    (stroke (width 0) (type default) (color 0 0 0 0))
+  )
+  (polyline (pts (xy 172.72 83.82) (xy 172.72 198.12))
     (stroke (width 0) (type default) (color 0 0 0 0))
   )
@@
     (stroke (width 0) (type default) (color 0 0 0 0))
   )
+  (polyline (pts (xy 20.32 83.82) (xy 20.32 198.12))
+    (stroke (width 0) (type default) (color 0 0 0 0))
+  )
   (wire (pts (xy 64.77 129.54) (xy 64.77 119.38))
     (stroke (width 0) (type default) (color 0 0 0 0))
@@
     (stroke (width 0) (type default) (color 0 0 0 0))
   )
+  (polyline (pts (xy 147.32 15.24) (xy 17.78 15.24))
+    (stroke (width 0) (type default) (color 0 0 0 0))
+  )
   (wire (pts (xy 146.812 218.44) (xy 136.652 218.44))
     (stroke (width 0) (type default) (color 0 0 0 0))
@@
   )
   (wire (pts (xy 97.282 266.573) (xy 97.282 271.653))
+    (stroke (width 0) (type default) (color 0 0 0 0))
+  )
+  (polyline (pts (xy 147.32 81.28) (xy 147.32 15.24))
     (stroke (width 0) (type default) (color 0 0 0 0))
   )
@@
     (effects (font (size 3.27 3.27) (thickness 0.654) bold) (justify left bottom))
   )
+  (label "SDA" (at 76.2 152.4 0)
+    (effects (font (size 1.27 1.27)) (justify left bottom))
+  )
   (label "SCL_3.3" (at 185.293 38.1 180)
     (effects (font (size 1.27 1.27) (thickness 0.254) bold) (justify right bottom))
@@
     (effects (font (size 1.27 1.27) bold) (justify left bottom))
   )
-  (label "RXD" (at 162.56 106.68 0)
+  (label "RXD" (at 162.56 109.22 0)
     (effects (font (size 1.27 1.27)) (justify left bottom))
   )
@@
     (effects (font (size 1.27 1.27) bold) (justify left bottom))
   )
+  (label "SCL" (at 76.2 154.94 0)
+    (effects (font (size 1.27 1.27)) (justify left bottom))
+  )
   (label "GND" (at 137.16 215.9 0)
     (effects (font (size 1.27 1.27) (thickness 0.254) bold) (justify left bottom))
@@
     (effects (font (size 1.27 1.27) bold) (justify left bottom))
   )
-  (label "TXD" (at 162.56 109.22 0)
+  (label "TXD" (at 162.56 106.68 0)
     (effects (font (size 1.27 1.27)) (justify left bottom))
   )
@@
       (effects (font (size 1.27 1.27)) (justify left))
     )
-    (property "Footprint" "" (id 2) (at 378.46 204.47 0)
+    (property "Footprint" "Crystal:Crystal_SMD_0603-4Pin_6.0x3.5mm" (id 2) (at 378.46 204.47 0)
       (effects (font (size 1.27 1.27)) hide)
     )
@@
   (symbol (lib_id "TP4056:TP4056") (at 112.522 248.793 0) (unit 1)
     (in_bom yes) (on_board yes) (fields_autoplaced)
-    (property "Reference" "U5" (id 0) (at 112.522 231.013 0))
-    (property "Value" "TP4056" (id 1) (at 112.522 233.553 0))
-    (property "Footprint" "tp4056 ftprnt:SOP127P600X175-9N" (id 2) (at 112.522 248.793 0)
+    (property "Reference" "U5" (id 0) (at 112.522 231.14 0))
+    (property "Value" "TP4056" (id 1) (at 112.522 233.68 0))
+    (property "Footprint" "Package_SO:SO-8_5.3x6.2mm_P1.27mm" (id 2) (at 112.522 248.793 0)
       (effects (font (size 1.27 1.27)) (justify left bottom) hide)
     )
@@
     )
     (path "/962f53be-4796-4882-97a5-e23946b557e2"
-      (reference "U5") (unit 1) (value "TP4056") (footprint "tp4056 ftprnt:SOP127P600X175-9N")
+      (reference "U5") (unit 1) (value "TP4056") (footprint "Package_SO:SO-8_5.3x6.2mm_P1.27mm")
     )
     (path "/819d13fc-46d6-4218-80e5-2fe7ce2c66df"
@@
     )
     (path "/47950098-5aec-4368-83a1-2986d2f1cf02"
-      (reference "Y1") (unit 1) (value "16MHZ") (footprint "")
-    )
-  )
+      (reference "Y1") (unit 1) (value "16MHZ") (footprint "Crystal:Crystal_SMD_0603-4Pin_6.0x3.5mm")
+    )
+  )

Commit message: add render folder
kicad 3d render image folder add
Parts:
- removed SW1: SW_SPDT, Button_Switch_SMD:SW_SPDT_PCM12, symbol Switch:SW_SPDT
Connections:
- net BATTERY +VE is gone; now on net VCC: C12.1 (P$1), J2.1 (Pin_1), U5.5 (BAT)
- no-connect marks 25 -> 24
Other:
- moved on the sheet: C10, C11, C9, R6, U4
